File: pcb/battery-manager/battery-manager.sch (KiCad schematic (older format))
At the start: 26 parts, among them J1 Conn_01x05_Female, J10 JST_2MM_MALE, J2 Conn_01x04_Female, J3 Conn_01x04_Female, J4 Conn_01x04_Female, J5 Conn_01x04_Female, J6 Conn_01x04_Female, J7 Conn_01x04_Female, J8 Conn_01x04_Female, J9 JST_2MM_MALE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

Commit message: pcb: update battery shield pcb to latest version
mainly, add a power path to supply the target with power when the
TP5400 is charging the battery, as in this mode the boost converter is
not active and the target is supplied with the current battery voltage
Parts:
- added D4: SS32, Diode_SMD:D_SMA, symbol Device:D_Schottky_Small
- added R4: 5k, Resistor_SMD:R_0805_2012Metric, symbol Device:R_Small
- J10, J9: symbol SparkFun-Connectors:JST_2MM_MALE -> battery-manager-rescue:JST_2MM_MALE-SparkFun-Connectors
- U1: symbol project:TP5400 -> battery-manager-rescue:TP5400-project
Connections:
- net GND: now also R4.2
- net USB_VBUS: now also D4.2 (A), R4.1
- net VOUT: now also D4.1 (K)
Changed lines of the file:
@@
 $EndDescr
 $Comp
-L project:TP5400 U1
+L battery-manager-rescue:TP5400-project U1
 U 1 1 5C6D3A5C
 P 5600 3050
@@
 VCC
 $Comp
-L SparkFun-Connectors:JST_2MM_MALE J9
+L battery-manager-rescue:JST_2MM_MALE-SparkFun-Connectors J9
 U 1 1 5C719919
 P 8900 3850
@@
 BAT
 $Comp
-L SparkFun-Connectors:JST_2MM_MALE J10
+L battery-manager-rescue:JST_2MM_MALE-SparkFun-Connectors J10
 U 1 1 5C7237C7
 P 8900 4550
@@
 $EndComp
 $Comp
-L power:PWR_FLAG #FLG?
+L power:PWR_FLAG #FLG0103
 U 1 1 5C78BB92
 P 1600 5900
-F 0 "#FLG?" H 1600 5975 50  0001 C CNN
+F 0 "#FLG0103" H 1600 5975 50  0001 C CNN
 F 1 "PWR_FLAG" H 1600 6074 50  0000 C CNN
 F 2 "" H 1600 5900 50  0001 C CNN
@@
 	1600 5900 1850 5900
 Connection ~ 1850 5900
+$Comp
+L Device:D_Schottky_Small D4
+U 1 1 5C7FE7C4
+P 4200 1600
+F 0 "D4" H 4200 1700 50  0000 C CNN
+F 1 "SS32" H 4000 1700 50  0000 C CNN
+F 2 "Diode_SMD:D_SMA" V 4200 1600 50  0001 C CNN
+F 3 "~" V 4200 1600 50  0001 C CNN
+	1    4200 1600
+	-1   0    0    1
+$EndComp
+Wire Wire Line
+	3700 1600 4000 1600
+Wire Wire Line
+	4550 1600 4300 1600
+Text Label 3700 1600 0    50   ~ 0
+USB_VBUS
+Text Label 4350 1600 0    50   ~ 0
+VOUT
+$Comp
+L Device:R_Small R4
+U 1 1 5C8050B2
+P 4000 1900
+F 0 "R4" H 4059 1946 50  0000 L CNN
+F 1 "5k" H 4059 1855 50  0000 L CNN
+F 2 "Resistor_SMD:R_0805_2012Metric" H 4000 1900 50  0001 C CNN
+F 3 "~" H 4000 1900 50  0001 C CNN
+	1    4000 1900
+	1    0    0    -1
+$EndComp
+$Comp
+L power:GND #PWR0115
+U 1 1 5C808A38
+P 4000 2100
+F 0 "#PWR0115" H 4000 1850 50  0001 C CNN
+F 1 "GND" H 4005 1927 50  0000 C CNN
+F 2 "" H 4000 2100 50  0001 C CNN
+F 3 "" H 4000 2100 50  0001 C CNN
+	1    4000 2100
+	1    0    0    -1
+$EndComp
+Wire Wire Line
+	4000 1600 4000 1800
+Connection ~ 4000 1600
+Wire Wire Line
+	4000 1600 4100 1600
+Wire Wire Line
+	4000 2000 4000 2100
 $EndSCHEMATC
